Commit message: 俯瞰カメラの実装

File: urdf/mmx7.xacro (robot description, xacro)
@@ -8,4 +8,5 @@
   <xacro:include filename="$(find crane_x7_description)/urdf/crane_x7.xacro" />
   <xacro:include filename="$(find kachaka_base_description)/urdf/kachaka_base.xacro" />
+  <xacro:include filename="$(find mmx7_description)/urdf/utils/global_camera_mounter.xacro" />
   <!-- <xacro:include filename="$(find orbbec_astra_camera)/urdf/astra.urdf.xacro" /> -->
   <xacro:macro name="mmx7"
@@ -203,5 +204,12 @@
       joint_hand_lower_limit="${joint_hand_lower_limit}"
       joint_hand_upper_limit="${joint_hand_upper_limit}" />
-    <link name="orbbec_mounting_branch_link">
+    <!-- 俯瞰カメラ -->
+    <xacro:global_camera_mounter />
+    <joint name="pedestal_to_orbbec_mounting_branch_joint" type="fixed">
+      <parent link="pedestal_link" />
+      <child link="vertical_branch_link" />
+      <origin xyz="0.010 0.085 -0.003" rpy="0 0 0" />
+    </joint>
+    <!-- <link name="orbbec_mounting_branch_link">
       <visual>
         <origin xyz="0 0 0.300" rpy="0 0 0" />
@@ -241,5 +249,5 @@
       <child link="orbbec_mounting_box_link" />
       <origin xyz="0.040 0 0.600" rpy="0 0 0" />
-    </joint>
+    </joint> -->
     <!--
     <xacro:astra parent="orbbec_mounting_box_link">

Commit message: プレート衝突実装忘れ

File: urdf/mmx7.xacro (robot description, xacro)
@@ -116,4 +116,10 @@
         <material name="silver" />
       </visual>
+      <collision>
+        <origin xyz="0 0 -0.0025" />
+        <geometry>
+          <box size="0.150 0.150 0.005" />
+        </geometry>
+      </collision>
     </link>
     <joint name="pedestal_link_to_mounting_plate_joint" type="fixed">
@@ -186,4 +192,5 @@
       <xacro:include filename="$(find realsense2_description)/urdf/_d435.urdf.xacro" />
       <xacro:sensor_d435
+        name="realsense_d435_camera"
         parent="${name_link_7}"
         use_nominal_extrinsics="false"

Commit message: 接触する不具合を解決

File: urdf/mmx7.xacro (robot description, xacro)
@@ -92,5 +92,5 @@
         <origin xyz="0 0 -0.182" rpy="0 0 0" />
         <geometry>
-          <box size="0.310 0.330 0.364" />
+          <box size="0.310 0.327 0.364" />
         </geometry>
         <material name="black" />
@@ -99,5 +99,5 @@
         <origin xyz="0 0 -0.182" rpy="0 0 0" />
         <geometry>
-          <box size="0.310 0.330 0.364" />
+          <box size="0.310 0.327 0.364" />
         </geometry>
       </collision>
@@ -126,5 +126,5 @@
       <parent link="pedestal_link" />
       <child link="mmx7_mounting_plate" />
-      <origin xyz="0.073 -0.075 0.001" rpy="0 0 0" />
+      <origin xyz="0.073 -0.045 0.001" rpy="0 0 0" />
     </joint>
     <xacro:crane_x7_arm
@@ -216,5 +216,5 @@
       <parent link="pedestal_link" />
       <child link="vertical_branch_link" />
-      <origin xyz="0.010 0.085 -0.003" rpy="0 0 0" />
+      <origin xyz="0.005 0.0835 -0.003" rpy="0 0 0" />
     </joint>
     <!-- <link name="orbbec_mounting_branch_link">

Commit message: 不要な記述を削除、realsenseカメラの追加のtf配信を許可

File: urdf/mmx7.xacro (robot description, xacro)
@@ -9,5 +9,4 @@
   <xacro:include filename="$(find kachaka_base_description)/urdf/kachaka_base.xacro" />
   <xacro:include filename="$(find mmx7_description)/urdf/utils/global_camera_mounter.xacro" />
-  <!-- <xacro:include filename="$(find orbbec_astra_camera)/urdf/astra.urdf.xacro" /> -->
   <xacro:macro name="mmx7"
     params="
@@ -194,5 +193,5 @@
         name="realsense_d435_camera"
         parent="${name_link_7}"
-        use_nominal_extrinsics="false"
+        use_nominal_extrinsics="true"
         add_plug="false"
         use_mesh="true">
@@ -218,47 +217,4 @@
       <origin xyz="0.005 0.0835 -0.003" rpy="0 0 0" />
     </joint>
-    <!-- <link name="orbbec_mounting_branch_link">
-      <visual>
-        <origin xyz="0 0 0.300" rpy="0 0 0" />
-        <geometry>
-          <box size="0.03 0.03 0.600" />
-        </geometry>
-        <material name="white" />
-      </visual>
-      <collision>
-        <origin xyz="0 0 0.300" rpy="0 0 0" />
-        <geometry>
-          <box size="0.03 0.03 0.600" />
-        </geometry>s </collision>
-    </link>
-    <joint name="pedestal_to_orbbec_mounting_branch_joint" type="fixed">
-      <parent link="pedestal_link" />
-      <child link="orbbec_mounting_branch_link" />
-      <origin xyz="0.010 0.085 -0.003" rpy="0 0 0" />
-    </joint>
-    <link name="orbbec_mounting_box_link">
-      <visual>
-        <origin xyz="0 0 -0.035" rpy="0 0 0" />
-        <geometry>
-          <box size="0.050 0.060 0.070" />
-        </geometry>
-        <material name="black" />
-      </visual>
-      <collision>
-        <origin xyz="0 0 -0.035" rpy="0 0 0" />
-        <geometry>
-          <box size="0.050 0.060 0.070" />
-        </geometry>
-      </collision>
-    </link>
-    <joint name="orbbec_mounting_branch_to_orbbec_mounting_box_joint" type="fixed">
-      <parent link="orbbec_mounting_branch_link" />
-      <child link="orbbec_mounting_box_link" />
-      <origin xyz="0.040 0 0.600" rpy="0 0 0" />
-    </joint> -->
-    <!--
-    <xacro:astra parent="orbbec_mounting_box_link">
-      <origin xyz="0 0 0" rpy="0 0 0" />
-    </xacro:astra> -->
   </xacro:macro>
 </robot>

File: urdf/utils/calibration_camera_mounter.xacro (robot description, xacro)
@@ -21,9 +21,4 @@
             </collision>
         </link>
-        <!-- <joint name="pedestal_to_orbbec_mounting_branch_joint" type="fixed">
-            <parent link="pedestal_link" />
-            <child link="vertical_branch_link" />
-            <origin xyz="0.010 0.085 -0.003" rpy="0 0 0" />
-        </joint> -->
         <xacro:micon_xl430_mounter />
         <joint name="branch_to_micon_xl430_joint" type="fixed">

File: urdf/utils/fixed_camera_mounter.xacro (robot description, xacro)
@@ -21,9 +21,4 @@
             </collision>
         </link>
-        <!-- <joint name="pedestal_to_orbbec_mounting_branch_joint" type="fixed">
-            <parent link="pedestal_link" />
-            <child link="vertical_branch_link" />
-            <origin xyz="0.010 0.085 -0.003" rpy="0 0 0" />
-        </joint> -->
         <xacro:micon_xl430_mounter />
         <joint name="branch_to_micon_xl430_joint" type="fixed">

File: urdf/utils/global_camera_mounter.xacro (robot description, xacro)
@@ -21,9 +21,4 @@
             </collision>
         </link>
-        <!-- <joint name="pedestal_to_orbbec_mounting_branch_joint" type="fixed">
-            <parent link="pedestal_link" />
-            <child link="vertical_branch_link" />
-            <origin xyz="0.010 0.085 -0.003" rpy="0 0 0" />
-        </joint> -->
         <xacro:micon_xl430_mounter />
         <joint name="branch_to_micon_xl430_joint" type="fixed">

File: urdf/utils/micon_xl430_mounter.xacro (robot description, xacro)
@@ -2,5 +2,4 @@
 <robot name="micon_xl430_mounter" xmlns:xacro="http://ros.org/wiki/xacro">
     <xacro:macro name="micon_xl430_mounter">
-        <!-- マウンタの下に設置されたマイコンも一つのマウンタとして宣言する -->
         <link name="micon_2xl430_mounter_link">
             <visual>

Commit message: 物理仕様の追加（動作未確認)

File: urdf/mmx7.xacro (robot description, xacro)
@@ -88,4 +88,9 @@
     </joint>
     <link name="pedestal_link">
+        <inertial>
+            <mass value="99.6" />
+            <origin xyz="0 0 -0.182" rpy="0 0 0" />
+            <inertia ixx="1.98" ixy="0.0" ixz="0.0" iyy="1.89" iyz="0.0" izz="1.68" />
+        </inertial>
       <visual>
         <origin xyz="0 0 -0.182" rpy="0 0 0" />
@@ -108,4 +113,9 @@
     </joint>
     <link name="mmx7_mounting_plate">
+        <inertial>
+            <mass value="0.30" />
+            <origin xyz="0 0 -0.0025" rpy="0 0 0" />
+            <inertia ixx="0.00056" ixy="0.0" ixz="0.0" iyy="0.00056" iyz="0.0" izz="0.00113" />
+        </inertial>
       <visual>
         <origin xyz="0 0 -0.0025" />

File: urdf/utils/global_camera_mounter.xacro (robot description, xacro)
@@ -28,5 +28,5 @@
         </joint>
         <xacro:xl430 />
-        <joint name="micon_xl430_mounter_to_xl430_joint" type="revolute">
+        <joint name="micon_xl430_mounter_to_xl430_joint" type="fixed">
             <parent link="micon_2xl430_mounter_link" />
             <child link="xl430_link" />
@@ -36,5 +36,5 @@
         </joint>
         <xacro:orbbec_mounter />
-        <joint name="xl430_to_orbbec_mounter_joint" type="revolute">
+        <joint name="xl430_to_orbbec_mounter_joint" type="fixed">
             <parent link="xl430_link" />
             <child link="orbbec_mounter_link" />
